Commit message: adding rviz and robot model publisher

File: coppeliasim_simulation/urdf_from_coppelia/twip.urdf (robot description, URDF)
Before this commit: robot body__32__, 3 links, 2 joints
Links:
- link Wheel1__34__: geometry collision cylinder length=0.029999999329448 radius=0.10000000149012; visual cylinder length=0.029999999329448 radius=0.10000000149012
- link Wheel2__36__: geometry collision cylinder length=0.029999999329448 radius=0.10000001639128; visual cylinder length=0.029999999329448 radius=0.10000000149012
- link body__32__: geometry collision box size=0.100000 0.200000 0.500000; visual box size=0.100000 0.200000 0.500000
